File: tutorial.kicad_pcb (KiCad board)
At the start: 2 copper layers, 85.2 x 38.1 mm, 24 parts, among them SW1 SW_Push, U1 ATmega32U4-AU, Y1 16MHz

Commit message: Fixes and cleanup
Parts:
- moved F1 2.07 mm to (67.4, 93.9)
- moved C3 0.52 mm to (88.6, 93.2)
- turned R1 to 270 degrees
Connections:
- C1 pad 2: +5V -> GND
- C2 pad 2: +5V -> GND
- C3 pad 2: +5V -> GND
- C4 pad 2: +5V -> GND
- C5 pad 2: +5V -> GND
- C6 pad 2: +5V -> GND
- C7 pad 2: +5V -> GND
- F1 pad 2: VCC -> +5V
- R4 pad 1: +5V -> GND
- SW1 pad 1: +5V -> GND
- U1 pad 15: +5V -> GND
- U1 pad 23: +5V -> GND
- U1 pad 35: +5V -> GND
- U1 pad 43: +5V -> GND
- U1 pad 5: +5V -> GND
- USB1 pad 1: +5V -> GND
- USB1 pad 5: VCC -> +5V
- Y1 pad 2: +5V -> GND
- Y1 pad 4: +5V -> GND
Other:
- board size 85.2 x 38.1 mm -> 85.1 x 38.1 mm
- net class Default: trace_width 0.25 -> 0.254
- net class Power added: clearance 0.2, trace_width 0.381, via_dia 0.8, via_drill 0.4

Commit message: Finished routing
Parts:
- moved C7 9.55 mm to (88.1, 97.8), turned to 270 degrees
- moved C3 2.75 mm to (88.9, 90.5)
- turned F1 to 90 degrees
Connections:
- F1 pad 2: +5V -> VCC
- U1 pad 27: Net-(U1-Pad27) -> ROW0
- U1 pad 28: Net-(U1-Pad28) -> COL1
- U1 pad 29: Net-(U1-Pad29) -> COL0
- U1 pad 30: Net-(U1-Pad30) -> ROW1
- USB1 pad 5: +5V -> VCC
Routing:
- net GND: track 0.00 -> 147.7 mm
- net +5V: track 0.00 -> 108.0 mm, vias 0 -> 5
- net COL1: track 0.00 -> 52.1 mm
- net ROW1: track 0.00 -> 51.5 mm
- net ROW0: track 0.00 -> 45.8 mm
- net Net-(R1-Pad2): track 0.00 -> 35.5 mm, vias 0 -> 2
- net COL0: track 0.00 -> 32.7 mm
- net Net-(R3-Pad1): track 0.00 -> 25.0 mm
- net Net-(R2-Pad1): track 0.00 -> 23.4 mm
- net Net-(C2-Pad1): track 0.00 -> 14.6 mm
- net VCC: track 0.00 -> 14.1 mm
- net Net-(C1-Pad1): track 0.00 -> 11.9 mm
- net Net-(D4-Pad2): track 0.00 -> 6.82 mm
- net Net-(D2-Pad2): track 0.00 -> 6.82 mm
- net Net-(D3-Pad2): track 0.00 -> 6.82 mm
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Other:
- net class Default: trace_width 0.254 -> 0.25
- net class Power: trace_width 0.381 -> 0.375
